File: pcb/DockPlatform/schematic.sch (EAGLE design)
At the start: 5 parts

Commit message: normal changes Pushed.
Parts:
- removed TRF1: T60403-K5024-X099, plc_lib:T60403-K5024-X099
- added R1: 1M,P1.0MACT-ND, SparkFun-Resistors:RESISTOR0805-RES
- added U$1: T60403-K5024-X099, plc_lib:T60403-K5024-X099
Connections:
- new net LINEA: R1.2, U$1.P$1
- new net LINENF: R1.1, U$1.P$2
- new net N$11: U$1.P$5, X2-1.KL, X2-2.KL
- net N$3: now also U$1.P$6
Other:
- note added: "PLC Transformer Coupling"
- moved on the sheet: C1, L1, X1-1, X1-2, X2-1, X2-2
